Commit message: added low poly stl files for better performance in simulation

File: akrobat/urdf/hexapod_high_poly.urdf (robot description, URDF)
Before this commit: robot hexapod, 20 links, 19 joints
Links:
- link 1_coxa_link: geometry visual mesh filename=package://akrobat/stl/high_poly/coxa_l_link.stl
- link 1_femur_link: geometry visual mesh filename=package://akrobat/stl/high_poly/femur_link.stl
- link 1_tibia_link: geometry visual mesh filename=package://akrobat/stl/high_poly/tibia_link.stl
- link 2_coxa_link: geometry visual mesh filename=package://akrobat/stl/high_poly/coxa_r_link.stl
- link 2_femur_link: geometry visual mesh filename=package://akrobat/stl/high_poly/femur_link.stl
- link 2_tibia_link: geometry visual mesh filename=package://akrobat/stl/high_poly/tibia_link.stl
- link 3_coxa_link: geometry visual mesh filename=package://akrobat/stl/high_poly/coxa_l_link.stl
- link 3_femur_link: geometry visual mesh filename=package://akrobat/stl/high_poly/femur_link.stl
- link 3_tibia_link: geometry visual mesh filename=package://akrobat/stl/high_poly/tibia_link.stl
- link 4_coxa_link: geometry visual mesh filename=package://akrobat/stl/high_poly/coxa_r_link.stl
- link 4_femur_link: geometry visual mesh filename=package://akrobat/stl/high_poly/femur_link.stl
- link 4_tibia_link: geometry visual mesh filename=package://akrobat/stl/high_poly/tibia_link.stl
- link 5_coxa_link: geometry visual mesh filename=package://akrobat/stl/high_poly/coxa_l_link.stl
- link 5_femur_link: geometry visual mesh filename=package://akrobat/stl/high_poly/femur_link.stl
- link 5_tibia_link: geometry visual mesh filename=package://akrobat/stl/high_poly/tibia_link.stl
- link 6_coxa_link: geometry visual mesh filename=package://akrobat/stl/high_poly/coxa_r_link.stl
- link 6_femur_link: geometry visual mesh filename=package://akrobat/stl/high_poly/femur_link.stl
- link 6_tibia_link: geometry visual mesh filename=package://akrobat/stl/high_poly/tibia_link.stl
- link hexapod_link: geometry visual mesh filename=package://akrobat/stl/high_poly/hexapod_link.stl
