Commit message: fixed xacro files to work with akrobat.rviz

File: akrobat/urdf/akrobat_high_poly.xacro (robot description, xacro)
@@ -12,5 +12,5 @@
 			<alwaysOn>true</alwaysOn>
 			<updateRate>30.0</updateRate>
-			<bodyName>base</bodyName>
+			<bodyName>base_link</bodyName>
 			<topicName>odom</topicName>
 			<gaussianNoise>0</gaussianNoise>
@@ -20,7 +20,7 @@
 		</plugin>
 	</gazebo>
-	<link name="base"/>
-	<joint name="base_to_akrobat_joint" type="fixed">
-		<parent link="base"/>
+	<link name="base_link"/>
+	<joint name="base_link_to_akrobat_joint" type="fixed">
+		<parent link="base_link"/>
 		<child link="akrobat_link"/>
 	</joint>

File: akrobat/urdf/akrobat_low_poly.xacro (robot description, xacro)
@@ -13,5 +13,5 @@
 			<alwaysOn>true</alwaysOn>
 			<updateRate>30.0</updateRate>
-			<bodyName>base</bodyName>
+			<bodyName>base_link</bodyName>
 			<topicName>odom</topicName>
 			<gaussianNoise>0</gaussianNoise>
@@ -21,7 +21,7 @@
 		</plugin>
 	</gazebo>
-	<link name="base"/>
-	<joint name="base_to_akrobat_joint" type="fixed">
-		<parent link="base"/>
+	<link name="base_link"/>
+	<joint name="base_link_to_akrobat_joint" type="fixed">
+		<parent link="base_link"/>
 		<child link="akrobat_link"/>
 	</joint>
