Commit message: updated xacro files to separate collision and visual geometry

File: akrobat/urdf/leg-1.xacro (robot description, xacro)
@@ -4,5 +4,5 @@
 		<visual>
 			<geometry>
-				<mesh filename="${stl_path}coxa_l_link.stl"/>
+				<mesh filename="${stl_path_visual}coxa_l_link.stl"/>
 			</geometry>
 			<origin rpy="0 0 0" xyz="0 0 0"/>
@@ -17,5 +17,5 @@
 		<collision>
 			<geometry>
-				<mesh filename="${stl_path}coxa_l_link.stl"/>
+				<mesh filename="${stl_path_collision}coxa_l_link.stl"/>
 			</geometry>
 			<origin rpy="0 0 0" xyz="0 0 0"/>
@@ -32,5 +32,5 @@
 		<visual>
 			<geometry>
-				<mesh filename="${stl_path}femur_link.stl"/>
+				<mesh filename="${stl_path_visual}femur_link.stl"/>
 			</geometry>
 			<origin rpy="0 0 0" xyz="0 0 0"/>
@@ -45,5 +45,5 @@
 		<collision>
 			<geometry>
-				<mesh filename="${stl_path}femur_link.stl"/>
+				<mesh filename="${stl_path_collision}femur_link.stl"/>
 			</geometry>
 			<origin rpy="0 0 0" xyz="0 0 0"/>
@@ -60,5 +60,5 @@
 		<visual>
 			<geometry>
-				<mesh filename="${stl_path}tibia_link.stl"/>
+				<mesh filename="${stl_path_visual}tibia_link.stl"/>
 			</geometry>
 			<origin rpy="0 0 0" xyz="0 0 0"/>
@@ -73,5 +73,5 @@
 		<collision>
 			<geometry>
-				<mesh filename="${stl_path}tibia_link.stl"/>
+				<mesh filename="${stl_path_collision}tibia_link.stl"/>
 			</geometry>
 			<origin rpy="0 0 0" xyz="0 0 0"/>

File: akrobat/urdf/leg-2.xacro (robot description, xacro)
@@ -4,5 +4,5 @@
 		<visual>
 			<geometry>
-				<mesh filename="${stl_path}coxa_r_link.stl"/>
+				<mesh filename="${stl_path_visual}coxa_r_link.stl"/>
 			</geometry>
 			<origin rpy="0 0 0" xyz="0 0 0"/>
@@ -17,5 +17,5 @@
 		<collision>
 			<geometry>
-				<mesh filename="${stl_path}coxa_r_link.stl"/>
+				<mesh filename="${stl_path_collision}coxa_r_link.stl"/>
 			</geometry>
 			<origin rpy="0 0 0" xyz="0 0 0"/>
@@ -32,5 +32,5 @@
 		<visual>
 			<geometry>
-				<mesh filename="${stl_path}femur_link.stl"/>
+				<mesh filename="${stl_path_visual}femur_link.stl"/>
 			</geometry>
 			<origin rpy="0 0 0" xyz="0 0 0"/>
@@ -45,5 +45,5 @@
 		<collision>
 			<geometry>
-				<mesh filename="${stl_path}femur_link.stl"/>
+				<mesh filename="${stl_path_collision}femur_link.stl"/>
 			</geometry>
 			<origin rpy="0 0 0" xyz="0 0 0"/>
@@ -60,5 +60,5 @@
 		<visual>
 			<geometry>
-				<mesh filename="${stl_path}tibia_link.stl"/>
+				<mesh filename="${stl_path_visual}tibia_link.stl"/>
 			</geometry>
 			<origin rpy="0 0 0" xyz="0 0 0"/>
@@ -73,5 +73,5 @@
 		<collision>
 			<geometry>
-				<mesh filename="${stl_path}tibia_link.stl"/>
+				<mesh filename="${stl_path_collision}tibia_link.stl"/>
 			</geometry>
 			<origin rpy="0 0 0" xyz="0 0 0"/>

File: akrobat/urdf/leg-3.xacro (robot description, xacro)
@@ -4,5 +4,5 @@
 		<visual>
 			<geometry>
-				<mesh filename="${stl_path}coxa_l_link.stl"/>
+				<mesh filename="${stl_path_visual}coxa_l_link.stl"/>
 			</geometry>
 			<origin rpy="0 0 0" xyz="0 0 0"/>
@@ -17,5 +17,5 @@
 		<collision>
 			<geometry>
-				<mesh filename="${stl_path}coxa_l_link.stl"/>
+				<mesh filename="${stl_path_collision}coxa_l_link.stl"/>
 			</geometry>
 			<origin rpy="0 0 0" xyz="0 0 0"/>
@@ -32,5 +32,5 @@
 		<visual>
 			<geometry>
-				<mesh filename="${stl_path}femur_link.stl"/>
+				<mesh filename="${stl_path_visual}femur_link.stl"/>
 			</geometry>
 			<origin rpy="0 0 0" xyz="0 0 0"/>
@@ -45,5 +45,5 @@
 		<collision>
 			<geometry>
-				<mesh filename="${stl_path}femur_link.stl"/>
+				<mesh filename="${stl_path_collision}femur_link.stl"/>
 			</geometry>
 			<origin rpy="0 0 0" xyz="0 0 0"/>
@@ -60,5 +60,5 @@
 		<visual>
 			<geometry>
-				<mesh filename="${stl_path}tibia_link.stl"/>
+				<mesh filename="${stl_path_visual}tibia_link.stl"/>
 			</geometry>
 			<origin rpy="0 0 0" xyz="0 0 0"/>
@@ -73,5 +73,5 @@
 		<collision>
 			<geometry>
-				<mesh filename="${stl_path}tibia_link.stl"/>
+				<mesh filename="${stl_path_collision}tibia_link.stl"/>
 			</geometry>
 			<origin rpy="0 0 0" xyz="0 0 0"/>

File: akrobat/urdf/leg-4.xacro (robot description, xacro)
@@ -4,5 +4,5 @@
 		<visual>
 			<geometry>
-				<mesh filename="${stl_path}coxa_r_link.stl"/>
+				<mesh filename="${stl_path_visual}coxa_r_link.stl"/>
 			</geometry>
 			<origin rpy="0 0 0" xyz="0 0 0"/>
@@ -17,5 +17,5 @@
 		<collision>
 			<geometry>
-				<mesh filename="${stl_path}coxa_r_link.stl"/>
+				<mesh filename="${stl_path_collision}coxa_r_link.stl"/>
 			</geometry>
 			<origin rpy="0 0 0" xyz="0 0 0"/>
@@ -32,5 +32,5 @@
 		<visual>
 			<geometry>
-				<mesh filename="${stl_path}femur_link.stl"/>
+				<mesh filename="${stl_path_visual}femur_link.stl"/>
 			</geometry>
 			<origin rpy="0 0 0" xyz="0 0 0"/>
@@ -45,5 +45,5 @@
 		<collision>
 			<geometry>
-				<mesh filename="${stl_path}femur_link.stl"/>
+				<mesh filename="${stl_path_collision}femur_link.stl"/>
 			</geometry>
 			<origin rpy="0 0 0" xyz="0 0 0"/>
@@ -60,5 +60,5 @@
 		<visual>
 			<geometry>
-				<mesh filename="${stl_path}tibia_link.stl"/>
+				<mesh filename="${stl_path_visual}tibia_link.stl"/>
 			</geometry>
 			<origin rpy="0 0 0" xyz="0 0 0"/>
@@ -73,5 +73,5 @@
 		<collision>
 			<geometry>
-				<mesh filename="${stl_path}tibia_link.stl"/>
+				<mesh filename="${stl_path_collision}tibia_link.stl"/>
 			</geometry>
 			<origin rpy="0 0 0" xyz="0 0 0"/>

File: akrobat/urdf/leg-5.xacro (robot description, xacro)
@@ -4,5 +4,5 @@
 		<visual>
 			<geometry>
-				<mesh filename="${stl_path}coxa_l_link.stl"/>
+				<mesh filename="${stl_path_visual}coxa_l_link.stl"/>
 			</geometry>
 			<origin rpy="0 0 0" xyz="0 0 0"/>
@@ -17,5 +17,5 @@
 		<collision>
 			<geometry>
-				<mesh filename="${stl_path}coxa_l_link.stl"/>
+				<mesh filename="${stl_path_collision}coxa_l_link.stl"/>
 			</geometry>
 			<origin rpy="0 0 0" xyz="0 0 0"/>
@@ -32,5 +32,5 @@
 		<visual>
 			<geometry>
-				<mesh filename="${stl_path}femur_link.stl"/>
+				<mesh filename="${stl_path_visual}femur_link.stl"/>
 			</geometry>
 			<origin rpy="0 0 0" xyz="0 0 0"/>
@@ -45,5 +45,5 @@
 		<collision>
 			<geometry>
-				<mesh filename="${stl_path}femur_link.stl"/>
+				<mesh filename="${stl_path_collision}femur_link.stl"/>
 			</geometry>
 			<origin rpy="0 0 0" xyz="0 0 0"/>
@@ -60,5 +60,5 @@
 		<visual>
 			<geometry>
-				<mesh filename="${stl_path}tibia_link.stl"/>
+				<mesh filename="${stl_path_visual}tibia_link.stl"/>
 			</geometry>
 			<origin rpy="0 0 0" xyz="0 0 0"/>
@@ -73,5 +73,5 @@
 		<collision>
 			<geometry>
-				<mesh filename="${stl_path}tibia_link.stl"/>
+				<mesh filename="${stl_path_collision}tibia_link.stl"/>
 			</geometry>
 			<origin rpy="0 0 0" xyz="0 0 0"/>

File: akrobat/urdf/leg-6.xacro (robot description, xacro)
@@ -4,5 +4,5 @@
 		<visual>
 			<geometry>
-				<mesh filename="${stl_path}coxa_r_link.stl"/>
+				<mesh filename="${stl_path_visual}coxa_r_link.stl"/>
 			</geometry>
 			<origin rpy="0 0 0" xyz="0 0 0"/>
@@ -17,5 +17,5 @@
 		<collision>
 			<geometry>
-				<mesh filename="${stl_path}coxa_r_link.stl"/>
+				<mesh filename="${stl_path_collision}coxa_r_link.stl"/>
 			</geometry>
 			<origin rpy="0 0 0" xyz="0 0 0"/>
@@ -32,5 +32,5 @@
 		<visual>
 			<geometry>
-				<mesh filename="${stl_path}femur_link.stl"/>
+				<mesh filename="${stl_path_visual}femur_link.stl"/>
 			</geometry>
 			<origin rpy="0 0 0" xyz="0 0 0"/>
@@ -45,5 +45,5 @@
 		<collision>
 			<geometry>
-				<mesh filename="${stl_path}femur_link.stl"/>
+				<mesh filename="${stl_path_collision}femur_link.stl"/>
 			</geometry>
 			<origin rpy="0 0 0" xyz="0 0 0"/>
@@ -60,5 +60,5 @@
 		<visual>
 			<geometry>
-				<mesh filename="${stl_path}tibia_link.stl"/>
+				<mesh filename="${stl_path_visual}tibia_link.stl"/>
 			</geometry>
 			<origin rpy="0 0 0" xyz="0 0 0"/>
@@ -73,5 +73,5 @@
 		<collision>
 			<geometry>
-				<mesh filename="${stl_path}tibia_link.stl"/>
+				<mesh filename="${stl_path_collision}tibia_link.stl"/>
 			</geometry>
 			<origin rpy="0 0 0" xyz="0 0 0"/>
