Commit message: added contact sensor plugin for tibia links

File: akrobat/urdf/akrobat.xacro (robot description, xacro)
@@ -9,4 +9,17 @@
 		</plugin>
 	</gazebo>
+	<xacro:macro name="contact_sensor_plugin" params="link_name">
+		<gazebo reference="${link_name}">
+            <sensor name="${link_name}_contact_sensor" type="contact">
+                <update_rate>10.0</update_rate>
+                <contact>
+                    <collision>${link_name}_collision</collision>
+                </contact>
+                <plugin name="${link_name}_contact_sensor_plugin" filename="libgazebo_ros_bumper.so">
+                    <bumperTopicName>leg_${link_name}_contact_sensor_state</bumperTopicName>
+                </plugin>
+            </sensor>
+        </gazebo>
+	</xacro:macro>
 	<link name="base_link"/>
 	<joint name="base_link_to_akrobat_joint" type="fixed">

File: akrobat/urdf/left_leg.xacro (robot description, xacro)
@@ -79,4 +79,5 @@
             </collision>
         </link>
+        <xacro:contact_sensor_plugin link_name="${leg_number}_tibia_link"/>
         <joint name="m${leg_number}3" type="revolute">
             <parent link="${leg_number}_femur_link"/>

File: akrobat/urdf/right_leg.xacro (robot description, xacro)
@@ -79,4 +79,5 @@
 			</collision>
 		</link>
+        <xacro:contact_sensor_plugin link_name="${leg_number}_tibia_link"/>
 		<joint name="m${leg_number}3" type="revolute">
 			<parent link="${leg_number}_femur_link"/>
