Commit message: recalculated inertia values for links

File: urdf/left_leg.xacro (robot description, xacro)
@@ -14,5 +14,5 @@
             <inertial>
                 <mass value="0.2"/>
-                <inertia ixx="4.99231E-05" ixy="7.69231E-08" ixz="0" iyy="4.83846E-05" iyz="0" izz="4.83846E-05"/>
+                <inertia ixx="82.2040461312" ixy="-3.1261621093999998e-06" ixz="-2.04e-14" iyy="85.2431273984" iyz="4e-16" izz="85.8957348864" />
             </inertial>
             <collision>
@@ -42,5 +42,5 @@
             <inertial>
                 <mass value="0.2"/>
-                <inertia ixx="2.40946E-05" ixy="-1.00676E-06" ixz="-7.43243E-07" iyy="0.000142824" iyz="-6.75676E-09" izz="0.000150466"/>
+                <inertia ixx="373.4843424768" ixy="-4.3218346e-09" ixz="-7.8324625e-05" iyy="2144.3060432896" iyz="-2.053010498e-07" izz="2269.8960879616" />
             </inertial>
             <collision>
@@ -70,5 +70,5 @@
             <inertial>
                 <mass value="0.2"/>
-                <inertia ixx="0.000296304" ixy="-4.34783E-08" ixz="3.26087E-06" iyy="0.000265391" iyz="1.73913E-06" izz="4.22174E-05"/>
+                <inertia ixx="677.4596304896" ixy="9.6555e-09" ixz="1.5286087649999998e-07" iyy="604.3930722304" iyz="6.896018065999999e-07" izz="98.687483904" />
             </inertial>
             <collision>

File: urdf/right_leg.xacro (robot description, xacro)
@@ -14,5 +14,5 @@
 			<inertial>
 				<mass value="0.2"/>
-				<inertia ixx="4.99231E-05" ixy="7.69231E-08" ixz="0" iyy="4.83846E-05" iyz="0" izz="4.83846E-05"/>
+				<inertia ixx="82.2065037312" ixy="-2.43e-14" ixz="1.63e-14" iyy="85.2328513536" iyz="-1e-16" izz="85.9001389056" />
 			</inertial>
 			<collision>
@@ -42,5 +42,5 @@
 			<inertial>
 				<mass value="0.2"/>
-				<inertia ixx="2.40946E-05" ixy="-1.00676E-06" ixz="-7.43243E-07" iyy="0.000142824" iyz="-6.75676E-09" izz="0.000150466"/>
+				<inertia ixx="373.4843424768" ixy="-4.3218346e-09" ixz="-7.8324625e-05" iyy="2144.3060432896" iyz="-2.053010498e-07" izz="2269.8960879616" />
 			</inertial>
 			<collision>
@@ -70,5 +70,5 @@
 			<inertial>
 				<mass value="0.2"/>
-				<inertia ixx="0.000296304" ixy="-4.34783E-08" ixz="3.26087E-06" iyy="0.000265391" iyz="1.73913E-06" izz="4.22174E-05"/>
+				<inertia ixx="677.4596304896" ixy="9.6555e-09" ixz="1.5286087649999998e-07" iyy="604.3930722304" iyz="6.896018065999999e-07" izz="98.687483904" />
 			</inertial>
 			<collision>
