Commit message: ros2_control WIP

File: urdf/akrobat.xacro (robot description, xacro)
@@ -4,11 +4,6 @@
 	<xacro:property name="stl_path_collision" value="file://$(find akrobat)/stl/collision/"/>
 	<xacro:property name="color_grey" value="0.67 0.67 0.67 1"/>
-	<gazebo>
-		<plugin filename="libgz_ros2_control-system.so" name="gz_ros2_control::GazeboSimROS2ControlPlugin">
-			<robot_param>robot_description</robot_param>
-			<robot_param_node>robot_state_publisher</robot_param_node>
-			<parameters>$(find akrobat)/config/akrobat_control.yaml</parameters>
-		</plugin>
-	</gazebo>
+	<xacro:arg name="simulation" default="False"/>
+	<xacro:include filename="$(find akrobat)/urdf/ros2_control.xacro"/>
 	<link name="world"/>
 	<joint name="world_to_akrobat_joint" type="fixed">

File: urdf/left_leg.xacro (robot description, xacro)
@@ -92,42 +92,4 @@
             <origin xyz="0 0.0 -0.162" rpy="0.0 0.0 0.0" />
         </joint>
-        <ros2_control name="GazeboSimSystem" type="system">
-            <hardware>
-                <plugin>gz_ros2_control/GazeboSimSystem</plugin>
-            </hardware>
-            <joint name="m${leg_number}1">
-                <command_interface name="effort">
-                    <param name="min">-1000</param>
-                    <param name="max">1000</param>
-                </command_interface>
-                <state_interface name="position">
-                    <param name="initial_value">0.0</param>
-                </state_interface>
-                <state_interface name="velocity"/>
-                <state_interface name="effort"/>
-            </joint>
-            <joint name="m${leg_number}2">
-                <command_interface name="effort">
-                    <param name="min">-1000</param>
-                    <param name="max">1000</param>
-                </command_interface>
-                <state_interface name="position">
-                    <param name="initial_value">0.0</param>
-                </state_interface>
-                <state_interface name="velocity"/>
-                <state_interface name="effort"/>
-            </joint>
-            <joint name="m${leg_number}3">
-                <command_interface name="effort">
-                    <param name="min">-1000</param>
-                    <param name="max">1000</param>
-                </command_interface>
-                <state_interface name="position">
-                    <param name="initial_value">0.0</param>
-                </state_interface>
-                <state_interface name="velocity"/>
-                <state_interface name="effort"/>
-            </joint>
-        </ros2_control>
     </xacro:macro>
 </robot>

File: urdf/right_leg.xacro (robot description, xacro)
@@ -92,42 +92,4 @@
 			<origin xyz="0 0.0 -0.162" rpy="0.0 0.0 0.0" />
 		</joint>
-		<ros2_control name="GazeboSimSystem" type="system">
-            <hardware>
-                <plugin>gz_ros2_control/GazeboSimSystem</plugin>
-            </hardware>
-            <joint name="m${leg_number}1">
-                <command_interface name="effort">
-                    <param name="min">-1000</param>
-                    <param name="max">1000</param>
-                </command_interface>
-                <state_interface name="position">
-                    <param name="initial_value">0.0</param>
-                </state_interface>
-                <state_interface name="velocity"/>
-                <state_interface name="effort"/>
-            </joint>
-            <joint name="m${leg_number}2">
-                <command_interface name="effort">
-                    <param name="min">-1000</param>
-                    <param name="max">1000</param>
-                </command_interface>
-                <state_interface name="position">
-                    <param name="initial_value">0.0</param>
-                </state_interface>
-                <state_interface name="velocity"/>
-                <state_interface name="effort"/>
-            </joint>
-            <joint name="m${leg_number}3">
-                <command_interface name="effort">
-                    <param name="min">-1000</param>
-                    <param name="max">1000</param>
-                </command_interface>
-                <state_interface name="position">
-                    <param name="initial_value">0.0</param>
-                </state_interface>
-                <state_interface name="velocity"/>
-                <state_interface name="effort"/>
-            </joint>
-        </ros2_control>
 	</xacro:macro>
 </robot>

Commit message: simulation progress

File: urdf/akrobat.xacro (robot description, xacro)
@@ -6,9 +6,4 @@
 	<xacro:arg name="simulation" default="False"/>
 	<xacro:include filename="$(find akrobat)/urdf/ros2_control.xacro"/>
-	<link name="world"/>
-	<joint name="world_to_akrobat_joint" type="fixed">
-		<parent link="world"/>
-		<child link="akrobat_link"/>
-	</joint>
 	<link name="akrobat_link">
 		<visual>

File: urdf/right_leg.xacro (robot description, xacro)
@@ -12,8 +12,8 @@
 				</material>
 			</visual>
-				<inertial>
-					<mass value="0.2"/>
-					<inertia ixx="4.99231E-05" ixy="7.69231E-08" ixz="0" iyy="4.83846E-05" iyz="0" izz="4.83846E-05"/>
-				</inertial>
+			<inertial>
+				<mass value="0.2"/>
+				<inertia ixx="4.99231E-05" ixy="7.69231E-08" ixz="0" iyy="4.83846E-05" iyz="0" izz="4.83846E-05"/>
+			</inertial>
 			<collision>
 				<geometry>

Commit message: major changes
xacro changed to make coordinate system follow ros conventions

tried to adjust inertia unsuccesfully

tripod gait implemented

File: urdf/akrobat.xacro (robot description, xacro)
@@ -4,4 +4,6 @@
 	<xacro:property name="stl_path_collision" value="file://$(find akrobat)/stl/collision/"/>
 	<xacro:property name="color_grey" value="0.67 0.67 0.67 1"/>
+	<xacro:property name="inertia_yaml" value="$(find akrobat)/urdf/inertia.yaml" />
+	<xacro:property name="inertia" value="${xacro.load_yaml(inertia_yaml)}" />
 	<xacro:arg name="simulation" default="False"/>
 	<xacro:include filename="$(find akrobat)/urdf/ros2_control.xacro"/>
@@ -11,5 +13,5 @@
 				<mesh filename="${stl_path_visual}hexapod_link.stl"/>
 			</geometry>
-			<origin rpy="0 0 0" xyz="0 0 0"/>
+			<origin rpy="0 0 ${pi/2}" xyz="0 0 0"/>
 			<material name="grey">
 				<color rgba="${color_grey}"/>
@@ -24,14 +26,13 @@
 				<mesh filename="${stl_path_collision}hexapod_link.stl"/>
 			</geometry>
-			<origin rpy="0 0 0" xyz="0 0 0"/>
+			<origin rpy="0 0 0" xyz="0 0 ${pi/2}"/>
 		</collision>
 	</link>
-	<xacro:include filename="$(find akrobat)/urdf/left_leg.xacro"/>
-	<xacro:include filename="$(find akrobat)/urdf/right_leg.xacro"/>
-	<xacro:left_leg leg_number="2" />
-	<xacro:left_leg leg_number="4" />
-	<xacro:left_leg leg_number="6" />
-	<xacro:right_leg leg_number="1" />
-	<xacro:right_leg leg_number="3" />
-	<xacro:right_leg leg_number="5" />
+	<xacro:include filename="$(find akrobat)/urdf/leg.xacro"/>
+	<xacro:leg leg_number="1" />
+	<xacro:leg leg_number="2" />
+	<xacro:leg leg_number="3" />
+	<xacro:leg leg_number="4" />
+	<xacro:leg leg_number="5" />
+	<xacro:leg leg_number="6" />
 </robot>
