Commit message: match urdf joint directions with real robot

File: urdf/leg.xacro (robot description, xacro)
@@ -36,5 +36,5 @@
 			<xacro:if value="${is_right_leg}">
 				<origin xyz="${(leg_number-4)/2*-0.217} 0.051 0" rpy="0 0 0"/>
-				<axis xyz="0 0 -1"/>
+				<axis xyz="0 0 1"/>
 			</xacro:if>
 			<xacro:unless value="${is_right_leg}">
@@ -49,9 +49,9 @@
 			<xacro:if value="${is_right_leg}">
 				<origin xyz="0 0.072 0" rpy="0 0 0"/>
-				<axis xyz="-1 0 0"/>
+				<axis xyz="1 0 0"/>
 			</xacro:if>
 			<xacro:unless value="${is_right_leg}">
 				<origin xyz="0 -0.072 0" rpy="0 0 0"/>
-				<axis xyz="1 0 0"/>
+				<axis xyz="-1 0 0"/>
 			</xacro:unless>
 			<limit effort="1000.0" lower="-3.14" upper="3.14" velocity="0.5"/>
@@ -62,9 +62,9 @@
 			<xacro:if value="${is_right_leg}">
 				<origin xyz="0 0.096 0" rpy="0 0 0"/>
-				<axis xyz="-1 0 0"/>
+				<axis xyz="1 0 0"/>
 			</xacro:if>
 			<xacro:unless value="${is_right_leg}">
 				<origin xyz="0 -0.096 0" rpy="0 0 0"/>
-				<axis xyz="1 0 0"/>
+				<axis xyz="-1 0 0"/>
 			</xacro:unless>
 			<limit effort="1000.0" lower="-3.14" upper="3.14" velocity="0.5"/>

Commit message: tripod gait adjusted

File: urdf/leg.xacro (robot description, xacro)
@@ -36,9 +36,9 @@
 			<xacro:if value="${is_right_leg}">
 				<origin xyz="${(leg_number-4)/2*-0.217} 0.051 0" rpy="0 0 0"/>
-				<axis xyz="0 0 1"/>
+				<axis xyz="0 0 -1"/>
 			</xacro:if>
 			<xacro:unless value="${is_right_leg}">
 				<origin xyz="${(leg_number-3)/2*-0.217} -0.051 0" rpy="0 0 0"/>
-				<axis xyz="0 0 1"/>
+				<axis xyz="0 0 -1"/>
 			</xacro:unless>
 			<limit effort="1000.0" lower="-3.14" upper="3.14" velocity="0.5"/>
